File: OrangePi_Zero3W_UPS_RevA.kicad_pcb (KiCad board)
At the start: 2 copper layers, 65 x 32 mm, 5 parts

Commit message: update phase 5A.1
Parts:
- removed the REF** at (64.0, 74.9)
- added J1: ORANGE_PI_ZERO_3W_HEADER, Connector_PinSocket_2.54mm:PinSocket_2x20_P2.54mm_Vertical, F.Cu at (64.0, 74.9)
Other:
- copper layers 2 -> 4

Commit message: phase 5a.1 revision
Other:
- board text added: "IMPORTANT: J1 is a bottom-mounted female stacking socket. J1 pad numbering is mirrored by row relative to the Orange Pi top-side physical header numbering. J1.1 mates OPI pin 2 J1.2 mates OPI pin 1 J1.3 mates OPI pin 4 J1.4 mates OPI pin 3 ..."
- board text added: "J1 PAD 1 → OPI PHYSICAL PIN 2 J1 PAD 2 → OPI PHYSICAL PIN 1"
- board text removed: "VERIFY PIN 1"

Commit message: Update OrangePi_Zero3W_UPS_RevA.kicad_pcb
Parts:
- added C1: 100nF, Capacitor_SMD:C_0603_1608Metric, F.Cu at (73.6, 81.5)
- added R1: 4.7k, Resistor_SMD:R_0603_1608Metric, F.Cu at (73.6, 84.0)
- added R2: 4.7k, Resistor_SMD:R_0603_1608Metric, F.Cu at (73.6, 86.5)
- added U1: MAX17048G_T10, MAX17048G_T10:SON50P200X200X80-9N, F.Cu at (78.3, 82.0)

Commit message: phase 5A.2 revisi
Parts:
- moved R2 6.82 mm to (78.0, 81.3)
- moved C1 4.94 mm to (74.0, 86.4)
- moved U1 2.79 mm to (76.2, 83.9)
- moved R1 2.66 mm to (74.0, 81.3)
Changed lines of the file:
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@@
 	(footprint "Resistor_SMD:R_0603_1608Metric"
 		(layer "F.Cu")
-		(at 73.625 86.47)
+		(at 78.045 81.28)
 		(descr "Resistor SMD 0603 (1608 Metric), square (rectangular) end terminal, IPC-7351 nominal, (Body size source: IPC-SM-782 page 72, https://www.pcb-3d.com/wordpress/wp-content/uploads/ipc-sm-782a_amendment_1_and_2.pdf), generated with kicad-footprint-generator")
 		(tags "resistor")
@@
 	(footprint "Capacitor_SMD:C_0603_1608Metric"
 		(layer "F.Cu")
-		(at 73.625 81.45)
+		(at 73.975 86.38)
 		(descr "Capacitor SMD 0603 (1608 Metric), square (rectangular) end terminal, IPC-7351 nominal, (Body size source: IPC-SM-782 page 76, https://www.pcb-3d.com/wordpress/wp-content/uploads/ipc-sm-782a_amendment_1_and_2.pdf), generated with kicad-footprint-generator")
 		(tags "capacitor")
@@
 	(footprint "Resistor_SMD:R_0603_1608Metric"
 		(layer "F.Cu")
-		(at 73.625 83.96)
+		(at 73.975 81.32)
 		(descr "Resistor SMD 0603 (1608 Metric), square (rectangular) end terminal, IPC-7351 nominal, (Body size source: IPC-SM-782 page 72, https://www.pcb-3d.com/wordpress/wp-content/uploads/ipc-sm-782a_amendment_1_and_2.pdf), generated with kicad-footprint-generator")
 		(tags "resistor")
@@
 	(footprint "MAX17048G_T10:SON50P200X200X80-9N"
 		(layer "F.Cu")
-		(at 78.275 82.02)
+		(at 76.245 83.94)
 		(property "Reference" "U1"
 			(at 1.365 -2.017 0)

Commit message: phase 5B.1B
Parts:
- moved C1 0.70 mm to (74.6, 86.2)
- moved U1 0.13 mm to (76.2, 83.8)
Changed lines of the file:
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@@
 	(footprint "Capacitor_SMD:C_0603_1608Metric"
 		(layer "F.Cu")
-		(at 73.975 86.38)
+		(at 74.645 86.18)
 		(descr "Capacitor SMD 0603 (1608 Metric), square (rectangular) end terminal, IPC-7351 nominal, (Body size source: IPC-SM-782 page 76, https://www.pcb-3d.com/wordpress/wp-content/uploads/ipc-sm-782a_amendment_1_and_2.pdf), generated with kicad-footprint-generator")
 		(tags "capacitor")
@@
 	(footprint "MAX17048G_T10:SON50P200X200X80-9N"
 		(layer "F.Cu")
-		(at 76.245 83.94)
+		(at 76.215 83.81)
 		(property "Reference" "U1"
-			(at 1.365 -2.017 0)
-			(layer "F.SilkS")
-			(effects
+			(at 2.495 0.14 0)
+			(layer "F.SilkS")
+			(effects
