File: OrangePi_Zero3W_UPS_RevA_before_silkscreen_cleanup.kicad_pcb (KiCad board)
At the start: 4 copper layers, 65 x 32 mm, 74 parts, among them J1 ORANGE_PI_ZERO_3W_HEADER, J2 BATTERY_1S_PROTECTED_NTC, J3 USB_C_POWER_INPUT, Q1 STL9P3LLH6, SW1 POWER / QON, U1 MAX17048G_T10, U2 BQ25895RTWR, U3 STUSB4500LQTR, U4 USBLC6-2SC6, U5 TPS61088RHLR, U6 TPS259470ARPWR

Commit message: warning cleaning
Other:
- board text added: "1u2"
- board text added: "2u2"
- board text added: "5V OUT"
- board text added: "BOOST"
- board text added: "CHARGE"
- board text added: "POWER"
- board text added: "UPS HAT • 5V / 3A"
- board text added: "USB IN"
- board text added: "USB-C"
- board text removed: "USB-C IN • CHARGER • BOOST • 5V OUT"
