File: OrangePi_Zero3W_UPS_RevA_before_power_placement.kicad_pcb (KiCad board)
At the start: 4 copper layers, 65 x 32 mm, 74 parts, among them J1 ORANGE_PI_ZERO_3W_HEADER, J2 BATTERY_1S_PROTECTED_NTC, J3 USB_C_POWER_INPUT, Q1 STL9P3LLH6, SW1 POWER / QON, U1 MAX17048G_T10, U2 BQ25895RTWR, U3 STUSB4500LQTR, U4 USBLC6-2SC6, U5 TPS61088RHLR, U6 TPS259470ARPWR

Commit message: Phase 6B.2B1: optimize BQ25895 charger power-loop placement
Parts:
- moved C3 1.21 mm to (87.5, 97.8)
- moved C4 1.21 mm to (91.5, 97.8)
- turned U2 to 0 degrees
Changed lines of the file:
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@@
 	(footprint "BQ25895RTWR:QFN50P400X400X80-25N"
 		(layer "F.Cu")
-		(at 82 89.815 -90)
+		(at 82 89.815)
 		(property "Reference" "U2"
-			(at -3.065 0.25 0)
+			(at 0.175 -3.635 0)
 			(layer "F.SilkS")
 			(effects
@@
 		)
 		(property "Value" "BQ25895RTWR"
-			(at 9.7 3.635 90)
+			(at 9.7 3.635 0)
 			(layer "F.Fab")
 			(effects
@@
 		)
 		(property "Datasheet" ""
-			(at 0 0 90)
+			(at 0 0 0)
 			(layer "F.Fab")
 			(hide yes)
@@
 		)
 		(property "Description" ""
-			(at 0 0 90)
+			(at 0 0 0)
 			(layer "F.Fab")
 			(hide yes)
@@
 		)
 		(property "MF" "Texas Instruments"
-			(at 0 0 270)
+			(at 0 0 0)
 			(unlocked yes)
 			(layer "F.Fab")
@@
 		)
 		(property "Description_1" "I2C 1cell 5A buck battery charger with high input voltage and 3.1-A boost with HVDCP enabled"
-			(at 0 0 270)
+			(at 0 0 0)
 			(unlocked yes)
 			(layer "F.Fab")
@@
 		)
 		(property "Package" "WQFN-24 Texas Instruments"
-			(at 0 0 270)
+			(at 0 0 0)
 			(unlocked yes)
 			(layer "F.Fab")
@@
 		)
 		(property "Price" "None"
-			(at 0 0 270)
+			(at 0 0 0)
 			(unlocked yes)
 			(layer "F.Fab")
@@
 		)
 		(property "SnapEDA_Link" "https://www.snapeda.com/parts/BQ25895RTWR/Texas+Instruments/view-part/?ref=snap"
-			(at 0 0 270)
+			(at 0 0 0)
 			(unlocked yes)
 			(layer "F.Fab")
@@
 		)
 		(property "MPN" "BQ25895RTWR"
-			(at 0 0 270)
+			(at 0 0 0)
 			(unlocked yes)
 			(layer "F.Fab")
@@
 		)
 		(property "Availability" "In Stock"
-			(at 0 0 270)
+			(at 0 0 0)
 			(unlocked yes)
 			(layer "F.Fab")
@@
 		)
 		(property "Check_prices" "https://www.snapeda.com/parts/BQ25895RTWR/Texas+Instruments/view-part/?ref=eda"
-			(at 0 0 270)
+			(at 0 0 0)
 			(unlocked yes)
 			(layer "F.Fab")
@@
 		)
 		(property "MP" "BQ25895RTWR"
-			(at 0 0 270)
+			(at 0 0 0)
 			(unlocked yes)
 			(layer "F.Fab")
@@
 		(attr smd)
 		(fp_line
-			(start -2 2)
-			(end -1.705 2)
+			(start -2 -2)
+			(end -2 -1.705)
 			(stroke
 				(width 0.127)
@@
 		)
 		(fp_line
-			(start -2 2)
-			(end -2 1.705)
+			(start -2 -2)
+			(end -1.705 -2)
 			(stroke
 				(width 0.127)
@@
 		)
 		(fp_line
-			(start 2 2)
-			(end 1.705 2)
+			(start -2 2)
+			(end -2 1.705)
 			(stroke
 				(width 0.127)
@@
 		)
 		(fp_line
-			(start 2 2)
-			(end 2 1.705)
+			(start -2 2)
+			(end -1.705 2)
 			(stroke
 				(width 0.127)
@@
 		)
 		(fp_line
-			(start -2 -2)
-			(end -2 -1.705)
+			(start 2 -2)
+			(end 1.705 -2)
 			(stroke
 				(width 0.127)
@@
 		)
 		(fp_line
-			(start -2 -2)
-			(end -1.705 -2)
+			(start 2 -2)
+			(end 2 -1.705)
 			(stroke
 				(width 0.127)
@@
 		)
 		(fp_line
-			(start 2 -2)
-			(end 2 -1.705)
+			(start 2 2)
+			(end 1.705 2)
 			(stroke
 				(width 0.127)
@@
 		)
 		(fp_line
-			(start 2 -2)
-			(end 1.705 -2)
+			(start 2 2)
+			(end 2 1.705)
 			(stroke
 				(width 0.127)
@@
 		)
 		(fp_line
-			(start -2.615 2.615)
-			(end 2.615 2.615)
+			(start -2.615 -2.615)
+			(end 2.615 -2.615)
 			(stroke
 				(width 0.05)
@@
 		)
 		(fp_line
-			(start 2.615 2.615)
-			(end 2.615 -2.615)
+			(start -2.615 2.615)
+			(end 2.615 2.615)
 			(stroke
 				(width 0.05)
@@
 		)
 		(fp_line
-			(start -2.615 -2.615)
+			(start 2.615 2.615)
 			(end 2.615 -2.615)
 			(stroke
@@
 		)
 		(fp_line
-			(start 2 2)
-			(end -2 2)
+			(start 2 -2)
+			(end -2 -2)
 			(stroke
 				(width 0.127)
@@
 		(fp_line
 			(start 2 2)
-			(end 2 -2)
+			(end -2 2)
 			(stroke
 				(width 0.127)
@@
 		)
 		(fp_line
-			(start 2 -2)
-			(end -2 -2)
+			(start 2 2)
+			(end 2 -2)
 			(stroke
 				(width 0.127)
@@
 		)
 		(pad "1" smd roundrect
-			(at -1.935 -1.25 270)
+			(at -1.935 -1.25)
 			(size 0.86 0.27)
 			(layers "F.Cu" "F.Mask" "F.Paste")
@@
 		)
 		(pad "2" smd roundrect
-			(at -1.935 -0.75 270)
+			(at -1.935 -0.75)
 			(size 0.86 0.27)
 			(layers "F.Cu" "F.Mask" "F.Paste")
@@
 		)
 		(pad "3" smd roundrect
-			(at -1.935 -0.25 270)
+			(at -1.935 -0.25)
 			(size 0.86 0.27)
 			(layers "F.Cu" "F.Mask" "F.Paste")
@@
 		)
 		(pad "4" smd roundrect
-			(at -1.935 0.25 270)
+			(at -1.935 0.25)
 			(size 0.86 0.27)
 			(layers "F.Cu" "F.Mask" "F.Paste")
@@
 		)
 		(pad "5" smd roundrect
-			(at -1.935 0.75 270)
+			(at -1.935 0.75)
 			(size 0.86 0.27)
 			(layers "F.Cu" "F.Mask" "F.Paste")
@@
 		)
 		(pad "6" smd roundrect
-			(at -1.935 1.25 270)
+			(at -1.935 1.25)
 			(size 0.86 0.27)
 			(layers "F.Cu" "F.Mask" "F.Paste")
@@
 		)
 		(pad "7" smd roundrect
-			(at -1.25 1.935 270)
+			(at -1.25 1.935)
 			(size 0.27 0.86)
 			(layers "F.Cu" "F.Mask" "F.Paste")
@@
 		)
 		(pad "8" smd roundrect
-			(at -0.75 1.935 270)
+			(at -0.75 1.935)
 			(size 0.27 0.86)
 			(layers "F.Cu" "F.Mask" "F.Paste")
@@
 		)
 		(pad "9" smd roundrect
-			(at -0.25 1.935 270)
+			(at -0.25 1.935)
 			(size 0.27 0.86)
 			(layers "F.Cu" "F.Mask" "F.Paste")
@@
 		)
 		(pad "10" smd roundrect
-			(at 0.25 1.935 270)
+			(at 0.25 1.935)
 			(size 0.27 0.86)
 			(layers "F.Cu" "F.Mask" "F.Paste")
@@
 		)
 		(pad "11" smd roundrect
-			(at 0.75 1.935 270)
+			(at 0.75 1.935)
 			(size 0.27 0.86)
 			(layers "F.Cu" "F.Mask" "F.Paste")
@@
 		)
 		(pad "12" smd roundrect
-			(at 1.25 1.935 270)
+			(at 1.25 1.935)
 			(size 0.27 0.86)
 			(layers "F.Cu" "F.Mask" "F.Paste")
@@
 		)
 		(pad "13" smd roundrect
-			(at 1.935 1.25 270)
+			(at 1.935 1.25)
 			(size 0.86 0.27)
 			(layers "F.Cu" "F.Mask" "F.Paste")
@@
 		)
 		(pad "14" smd roundrect
-			(at 1.935 0.75 270)
+			(at 1.935 0.75)
 			(size 0.86 0.27)
 			(layers "F.Cu" "F.Mask" "F.Paste")
@@
 		)
 		(pad "15" smd roundrect
-			(at 1.935 0.25 270)
+			(at 1.935 0.25)
 			(size 0.86 0.27)
 			(layers "F.Cu" "F.Mask" "F.Paste")
@@
 		)
 		(pad "16" smd roundrect
-			(at 1.935 -0.25 270)
+			(at 1.935 -0.25)
 			(size 0.86 0.27)
 			(layers "F.Cu" "F.Mask" "F.Paste")
@@
 		)
 		(pad "17" smd roundrect
-			(at 1.935 -0.75 270)
+			(at 1.935 -0.75)
 			(size 0.86 0.27)
 			(layers "F.Cu" "F.Mask" "F.Paste")
@@
 		)
 		(pad "18" smd roundrect
-			(at 1.935 -1.25 270)
+			(at 1.935 -1.25)
 			(size 0.86 0.27)
 			(layers "F.Cu" "F.Mask" "F.Paste")
@@
 		)
 		(pad "19" smd roundrect
-			(at 1.25 -1.935 270)
+			(at 1.25 -1.935)
 			(size 0.27 0.86)
 			(layers "F.Cu" "F.Mask" "F.Paste")
@@
 		)
 		(pad "20" smd roundrect
-			(at 0.75 -1.935 270)
+			(at 0.75 -1.935)
 			(size 0.27 0.86)
 			(layers "F.Cu" "F.Mask" "F.Paste")
@@
 		)
 		(pad "21" smd roundrect
-			(at 0.25 -1.935 270)
+			(at 0.25 -1.935)
 			(size 0.27 0.86)
 			(layers "F.Cu" "F.Mask" "F.Paste")
@@
 		)
 		(pad "22" smd roundrect
-			(at -0.25 -1.935 270)
+			(at -0.25 -1.935)
 			(size 0.27 0.86)
 			(layers "F.Cu" "F.Mask" "F.Paste")
@@
 		)
 		(pad "23" smd roundrect
-			(at -0.75 -1.935 270)
+			(at -0.75 -1.935)
 			(size 0.27 0.86)
 			(layers "F.Cu" "F.Mask" "F.Paste")
@@
 		)
 		(pad "24" smd roundrect
-			(at -1.25 -1.935 270)
+			(at -1.25 -1.935)
 			(size 0.27 0.86)
 			(layers "F.Cu" "F.Mask" "F.Paste")
@@
 		)
 		(pad "25" smd rect
-			(at 0 0 270)
+			(at 0 0)
 			(size 2.6 2.6)
 			(layers "F.Cu" "F.Mask")
@@
 	(footprint "Capacitor_SMD:C_0805_2012Metric"
 		(layer "F.Cu")
-		(at 92.2 96.75)
+		(at 91.52 97.75)
 		(descr "Capacitor SMD 0805 (2012 Metric), square (rectangular) end terminal, IPC-7351 nominal, (Body size source: IPC-SM-782 page 76, https://www.pcb-3d.com/wordpress/wp-content/uploads/ipc-sm-782a_amendment_1_and_2.pdf, https://docs.google.com/spreadsheets/d/1BsfQQcO9C6DZCsRaXUlFlo91Tg2WpOkGARC1WS5S8t0/edit?usp=sharing), generated with kicad-footprint-generator")
 		(tags "capacitor")
@@
 	(footprint "Capacitor_SMD:C_0805_2012Metric"
 		(layer "F.Cu")
-		(at 88.2 96.75)
+		(at 87.52 97.75)
 		(descr "Capacitor SMD 0805 (2012 Metric), square (rectangular) end terminal, IPC-7351 nominal, (Body size source: IPC-SM-782 page 76, https://www.pcb-3d.com/wordpress/wp-content/uploads/ipc-sm-782a_amendment_1_and_2.pdf, https://docs.google.com/spreadsheets/d/1BsfQQcO9C6DZCsRaXUlFlo91Tg2WpOkGARC1WS5S8t0/edit?usp=sharing), generated with kicad-footprint-generator")
 		(tags "capacitor")
